Commit message: applied pre-commits

File: sdf_contact_estimation_demo/urdf/ugv_base.urdf.xacro (robot description, xacro)
@@ -32,5 +32,5 @@
           <box size="${chassis_length_x} ${chassis_length_y} ${chassis_length_z}"/>
         </geometry>
-        <material name="MatteMetalicSlateBlue">
+        <material name="MatteMetallicSlateBlue">
           <color rgba="0 0.18 0.32 1"/>
         </material>
@@ -41,5 +41,5 @@
           <box size="${chassis_length_x} ${chassis_length_y} ${chassis_length_z}"/>
         </geometry>
-        <material name="MatteMetalicSlateBlue">
+        <material name="MatteMetallicSlateBlue">
           <color rgba="0 0.18 0.32 1"/>
         </material>
