Commit message: reformatting

File: sdf_contact_estimation_demo/urdf/tracked_robot.urdf.xacro (robot description, xacro)
@@ -1,4 +1,4 @@
 <?xml version="1.0"?>
-<robot name="tracked_robot" xmlns:xacro="http://www.ros.org/wiki/xacro">
+<robot xmlns:xacro="http://www.ros.org/wiki/xacro" name="tracked_robot">
   <!-- Included URDF Files -->
   <xacro:include filename="$(find sdf_contact_estimation_demo)/urdf/ugv_base.urdf.xacro"/>

File: sdf_contact_estimation_demo/urdf/ugv_base.urdf.xacro (robot description, xacro)
@@ -44,5 +44,5 @@
           <color rgba="0 0.18 0.32 1"/>
         </material>
-        </collision>
+      </collision>
     </link>
     <!-- Main tracks -->
@@ -54,8 +54,6 @@
     </xacro:main_track>
     <!-- Flippers -->
-    <xacro:flipper_pair name="flipper_front" parent="chassis_link" front="1"
-                                           x="${flipper_x_offset}" y="${flipper_y_offset}" z="${flipper_z_offset}" yaw="${pi}" pitch="${pi}"/>
-    <xacro:flipper_pair name="flipper_back" parent="chassis_link" front="-1"
-                                           x="${-flipper_x_offset}" y="${flipper_y_offset}" z="${flipper_z_offset}" pitch="${pi}"/>
+    <xacro:flipper_pair name="flipper_front" parent="chassis_link" front="1" x="${flipper_x_offset}" y="${flipper_y_offset}" z="${flipper_z_offset}" yaw="${pi}" pitch="${pi}"/>
+    <xacro:flipper_pair name="flipper_back" parent="chassis_link" front="-1" x="${-flipper_x_offset}" y="${flipper_y_offset}" z="${flipper_z_offset}" pitch="${pi}"/>
   </xacro:macro>
 </robot>
